Commit message: add feature-real

File: qm_description/urdf/qudraputed_manipulator/robot.urdf (robot description, URDF)
Before this commit: robot qm, 27 links, 26 joints
Links:
- added link camera_odom_frame
- link j2n6s300_link_1: geometry visual mesh filename=package://qm_description/meshes/manipulator/ring_big.dae; visual mesh filename=package://qm_description/meshes/manipulator/shoulder.dae
- link j2n6s300_link_2: geometry visual mesh filename=package://qm_description/meshes/manipulator/arm.dae; visual mesh filename=package://qm_description/meshes/manipulator/ring_big.dae
- link j2n6s300_link_3: geometry visual mesh filename=package://qm_description/meshes/manipulator/forearm.dae; visual mesh filename=package://qm_description/meshes/manipulator/ring_big.dae
- link j2n6s300_link_4: geometry visual mesh filename=package://qm_description/meshes/manipulator/ring_small.dae; visual mesh filename=package://qm_description/meshes/manipulator/wrist.dae
- link j2n6s300_link_5: geometry visual mesh filename=package://qm_description/meshes/manipulator/ring_small.dae; visual mesh filename=package://qm_description/meshes/manipulator/wrist.dae
- link j2n6s300_link_6: geometry visual mesh filename=package://qm_description/meshes/manipulator/hand_3finger.dae; visual mesh filename=package://qm_description/meshes/manipulator/ring_small.dae
- link j2n6s300_link_base: geometry visual mesh filename=package://qm_description/meshes/manipulator/base.dae
Joints:
- added joint camera_joint: type fixed, parent base, child camera_odom_frame, origin xyz=0.12 0.0 0.18 rpy=0.0 0.0 0.0

File: qm_description/urdf/qudraputed_manipulator/robot.xacro (robot description, xacro)
@@ -6,4 +6,11 @@
     <!-- manipulatior -->
     <xacro:include filename="$(find qm_description)/urdf/manipulator/j2n6s300fix.xacro"/>
+    <!-- camera -->
+    <link name="camera_pose_frame" />
+    <joint name="camera_joint" type="fixed">
+        <parent link= "base" />
+        <child link = "camera_pose_frame" />
+        <origin xyz="0.12 0.0 0.18" rpy="0.0 0.0 0.0" />
+    </joint>
     <link name="arm_base_link" />
     <joint name="manipulator_joint" type="fixed">

File: qm_description/urdf/qudraputed_manipulator/robot_mpc.xacro (robot description, xacro)
@@ -18,5 +18,5 @@
             <robotNamespace>/</robotNamespace>
             <robotParam>qm_description</robotParam>
-            <robotSimType>qm_gazebo/QMMpcHwSim</robotSimType>
+            <robotSimType>qm_gazebo/DogHwSim</robotSimType>
         </plugin>
     </gazebo>
