Commit message: add door world

File: qm_description/urdf/quadruped/aliengo.urdf (robot description, URDF)
Before this commit: robot qm, 27 links, 26 joints
Links:
- removed link arm_base_link
- removed link j2n6s300_end_effector
- removed link j2n6s300_link_1
- removed link j2n6s300_link_2
- removed link j2n6s300_link_3
- removed link j2n6s300_link_4
- removed link j2n6s300_link_5
- removed link j2n6s300_link_6
- removed link j2n6s300_link_base
- link LF_calf: geometry collision box size=0.25 0.0208 0.016; visual mesh filename=package://qm_description/meshes/quadruped/aliengo/calf.dae scale=1 1 1
- link LF_hip: geometry collision cylinder length=0.0418 radius=0.046; visual mesh filename=package://qm_description/meshes/quadruped/aliengo/hip.dae scale=1 1 1
- link LF_thigh: geometry collision box size=0.25 0.0374 0.043; collision cylinder length=0.03 radius=0.044
- link LH_calf: geometry collision box size=0.25 0.0208 0.016; visual mesh filename=package://qm_description/meshes/quadruped/aliengo/calf.dae scale=1 1 1
- link LH_hip: geometry collision cylinder length=0.0418 radius=0.046; visual mesh filename=package://qm_description/meshes/quadruped/aliengo/hip.dae scale=1 1 1
- link LH_thigh: geometry collision box size=0.25 0.0374 0.043; collision cylinder length=0.03 radius=0.044
- link RF_calf: geometry collision box size=0.25 0.0208 0.016; visual mesh filename=package://qm_description/meshes/quadruped/aliengo/calf.dae scale=1 1 1
- link RF_hip: geometry collision cylinder length=0.0418 radius=0.046; visual mesh filename=package://qm_description/meshes/quadruped/aliengo/hip.dae scale=1 1 1
- link RF_thigh: geometry collision box size=0.25 0.0374 0.043; collision cylinder length=0.03 radius=0.044
- link RH_calf: geometry collision box size=0.25 0.0208 0.016; visual mesh filename=package://qm_description/meshes/quadruped/aliengo/calf.dae scale=1 1 1
- link RH_hip: geometry collision cylinder length=0.0418 radius=0.046; visual mesh filename=package://qm_description/meshes/quadruped/aliengo/hip.dae scale=1 1 1
- link RH_thigh: geometry collision box size=0.25 0.0374 0.043; collision cylinder length=0.03 radius=0.044
- link base: geometry collision box size=0.647 0.15 0.112; visual mesh filename=package://qm_description/meshes/quadruped/aliengo/trunk.dae scale=1 1 1
Joints:
- removed joint j2n6s300_joint_1
- removed joint j2n6s300_joint_2
- removed joint j2n6s300_joint_3
- removed joint j2n6s300_joint_4
- removed joint j2n6s300_joint_5
- removed joint j2n6s300_joint_6
- removed joint j2n6s300_joint_base
- removed joint j2n6s300_joint_end_effector
- removed joint manipulator_joint

File: qm_description/urdf/quadruped/common/leg.xacro (robot description, xacro)
@@ -1,5 +1,5 @@
 <?xml version="1.0"?>
 <robot xmlns:xacro="http://www.ros.org/wiki/xacro">
-    <xacro:include filename="$(find qm_description)/urdf/qudraputed/common/transmission.xacro"/>
+    <xacro:include filename="$(find qm_description)/urdf/quadruped/common/transmission.xacro"/>
     <xacro:macro name="leg" params="prefix mirror mirror_dae front_hind front_hind_dae *origin">
         <joint name="${prefix}_HAA" type="revolute">
@@ -33,5 +33,5 @@
                 </xacro:if>
                 <geometry>
-                    <mesh filename="package://qm_description/meshes/qudraputed/$(arg robot_type)/hip.dae"
+                    <mesh filename="package://qm_description/meshes/quadruped/$(arg robot_type)/hip.dae"
                           scale="1 1 1"/>
                 </geometry>
@@ -67,9 +67,9 @@
                 <geometry>
                     <xacro:if value="${mirror_dae == True}">
-                        <mesh filename="package://qm_description/meshes/qudraputed/$(arg robot_type)/thigh.dae"
+                        <mesh filename="package://qm_description/meshes/quadruped/$(arg robot_type)/thigh.dae"
                               scale="1 1 1"/>
                     </xacro:if>
                     <xacro:if value="${mirror_dae == False}">
-                        <mesh filename="package://qm_description/meshes/qudraputed/$(arg robot_type)/thigh_mirror.dae"
+                        <mesh filename="package://qm_description/meshes/quadruped/$(arg robot_type)/thigh_mirror.dae"
                               scale="1 1 1"/>
                     </xacro:if>
@@ -110,5 +110,5 @@
                 <origin rpy="0 0 0" xyz="0 0 0"/>
                 <geometry>
-                    <mesh filename="package://qm_description/meshes/qudraputed/$(arg robot_type)/calf.dae"
+                    <mesh filename="package://qm_description/meshes/quadruped/$(arg robot_type)/calf.dae"
                           scale="1 1 1"/>
                 </geometry>

File: qm_description/urdf/quadruped/robot.xacro (robot description, xacro)
@@ -2,14 +2,14 @@
 <robot xmlns:xacro="http://www.ros.org/wiki/xacro" name="robot">
     <xacro:arg name="robot_type" default="aliengo"/>
-    <xacro:include filename="$(find qm_description)/urdf/qudraputed/common/materials.xacro"/>
-    <xacro:include filename="$(find qm_description)/urdf/qudraputed/common/leg.xacro"/>
-    <xacro:include filename="$(find qm_description)/urdf/qudraputed/common/gazebo.xacro"/>
-    <xacro:include filename="$(find qm_description)/urdf/qudraputed/common/imu.xacro"/>
-    <xacro:include filename="$(find qm_description)/urdf/qudraputed/$(arg robot_type)/const.xacro"/>
+    <xacro:include filename="$(find qm_description)/urdf/quadruped/common/materials.xacro"/>
+    <xacro:include filename="$(find qm_description)/urdf/quadruped/common/leg.xacro"/>
+    <xacro:include filename="$(find qm_description)/urdf/quadruped/common/gazebo.xacro"/>
+    <xacro:include filename="$(find qm_description)/urdf/quadruped/common/imu.xacro"/>
+    <xacro:include filename="$(find qm_description)/urdf/quadruped/$(arg robot_type)/const.xacro"/>
     <link name="base">
         <visual>
             <origin rpy="0 0 0" xyz="0 0 0"/>
             <geometry>
-                <mesh filename="package://qm_description/meshes/qudraputed/$(arg robot_type)/trunk.dae" scale="1 1 1"/>
+                <mesh filename="package://qm_description/meshes/quadruped/$(arg robot_type)/trunk.dae" scale="1 1 1"/>
             </geometry>
         </visual>

File: qm_description/urdf/quadruped_manipulator/robot.urdf (robot description, URDF)
Before this commit: robot robot, 18 links, 17 joints
Links:
- added link arm_base_link
- added link j2n6s300_end_effector
- added link j2n6s300_link_1, mass 0.7477; collision mesh filename=package://qm_description/meshes/manipulator/shoulder.dae; visual mesh filename=package://qm_description/meshes/manipulator/ring_big.dae
- added link j2n6s300_link_2, mass 0.99; collision mesh filename=package://qm_description/meshes/manipulator/arm.dae; visual mesh filename=package://qm_description/meshes/manipulator/arm.dae
- added link j2n6s300_link_3, mass 0.6763; collision mesh filename=package://qm_description/meshes/manipulator/forearm.dae; visual mesh filename=package://qm_description/meshes/manipulator/forearm.dae
- added link j2n6s300_link_4, mass 0.426367; collision mesh filename=package://qm_description/meshes/manipulator/wrist.dae; visual mesh filename=package://qm_description/meshes/manipulator/ring_small.dae
- added link j2n6s300_link_5, mass 0.426367; collision mesh filename=package://qm_description/meshes/manipulator/wrist.dae; visual mesh filename=package://qm_description/meshes/manipulator/ring_small.dae
- added link j2n6s300_link_6, mass 0.99; collision mesh filename=package://qm_description/meshes/manipulator/hand_3finger.dae; visual mesh filename=package://qm_description/meshes/manipulator/hand_3finger.dae
- added link j2n6s300_link_base, mass 0.46784; collision mesh filename=package://qm_description/meshes/manipulator/base.dae; visual mesh filename=package://qm_description/meshes/manipulator/base.dae
- link LF_calf: geometry collision box size=0.25 0.0208 0.016; visual mesh filename=package://qm_description/meshes/quadruped/aliengo/calf.dae scale=1 1 1
- link LF_hip: geometry collision cylinder length=0.0418 radius=0.046; visual mesh filename=package://qm_description/meshes/quadruped/aliengo/hip.dae scale=1 1 1
- link LF_thigh: geometry collision box size=0.25 0.0374 0.043; collision cylinder length=0.03 radius=0.044
- link LH_calf: geometry collision box size=0.25 0.0208 0.016; visual mesh filename=package://qm_description/meshes/quadruped/aliengo/calf.dae scale=1 1 1
- link LH_hip: geometry collision cylinder length=0.0418 radius=0.046; visual mesh filename=package://qm_description/meshes/quadruped/aliengo/hip.dae scale=1 1 1
- link LH_thigh: geometry collision box size=0.25 0.0374 0.043; collision cylinder length=0.03 radius=0.044
- link RF_calf: geometry collision box size=0.25 0.0208 0.016; visual mesh filename=package://qm_description/meshes/quadruped/aliengo/calf.dae scale=1 1 1
- link RF_hip: geometry collision cylinder length=0.0418 radius=0.046; visual mesh filename=package://qm_description/meshes/quadruped/aliengo/hip.dae scale=1 1 1
- link RF_thigh: geometry collision box size=0.25 0.0374 0.043; collision cylinder length=0.03 radius=0.044
- link RH_calf: geometry collision box size=0.25 0.0208 0.016; visual mesh filename=package://qm_description/meshes/quadruped/aliengo/calf.dae scale=1 1 1
- link RH_hip: geometry collision cylinder length=0.0418 radius=0.046; visual mesh filename=package://qm_description/meshes/quadruped/aliengo/hip.dae scale=1 1 1
- link RH_thigh: geometry collision box size=0.25 0.0374 0.043; collision cylinder length=0.03 radius=0.044
- link base: geometry collision box size=0.647 0.15 0.112; visual mesh filename=package://qm_description/meshes/quadruped/aliengo/trunk.dae scale=1 1 1
Joints:
- added joint j2n6s300_joint_1: type revolute, parent j2n6s300_link_base, child j2n6s300_link_1, origin xyz=0 0 0.15675 rpy=0 3.141592653589793 0, axis 0 0 1, limit lower=-6.283185307179586 upper=6.283185307179586 effort=40 velocity=0.6283185307179586
- added joint j2n6s300_joint_2: type revolute, parent j2n6s300_link_1, child j2n6s300_link_2, origin xyz=0 0.0016 -0.11875 rpy=-1.5707963267948966 0 3.141592653589793, axis 0 0 1, limit lower=0.8203047484373349 upper=5.462880558742252 effort=80 velocity=0.6283185307179586
- added joint j2n6s300_joint_3: type revolute, parent j2n6s300_link_2, child j2n6s300_link_3, origin xyz=0 -0.410 0 rpy=0 3.141592653589793 0, axis 0 0 1, limit lower=0.33161255787892263 upper=5.951572749300664 effort=40 velocity=0.6283185307179586
- added joint j2n6s300_joint_4: type revolute, parent j2n6s300_link_3, child j2n6s300_link_4, origin xyz=0 0.2073 -0.0114 rpy=-1.5707963267948966 0 3.141592653589793, axis 0 0 1, limit lower=-6.283185307179586 upper=6.283185307179586 effort=20 velocity=0.8377580409572781
- added joint j2n6s300_joint_5: type revolute, parent j2n6s300_link_4, child j2n6s300_link_5, origin xyz=0 -0.03703 -0.06414 rpy=1.0471975511965976 0 3.141592653589793, axis 0 0 1, limit lower=-6.283185307179586 upper=6.283185307179586 effort=20 velocity=0.8377580409572781
- added joint j2n6s300_joint_6: type revolute, parent j2n6s300_link_5, child j2n6s300_link_6, origin xyz=0 -0.03703 -0.06414 rpy=1.0471975511965976 0 3.141592653589793, axis 0 0 1, limit lower=-6.283185307179586 upper=6.283185307179586 effort=20 velocity=0.8377580409572781
- added joint j2n6s300_joint_base: type fixed, parent arm_base_link, child j2n6s300_link_base, origin xyz=0 0 0 rpy=0 0 0, axis 0 0 0
- added joint j2n6s300_joint_end_effector: type fixed, parent j2n6s300_link_6, child j2n6s300_end_effector, origin xyz=0 0 -0.1600 rpy=3.141592653589793 0 1.5707963267948966, axis 0 0 0
- added joint manipulator_joint: type fixed, parent base, child arm_base_link, origin xyz=0.0 0.0 0.01 rpy=0.0 0.0 0.0

File: qm_description/urdf/quadruped_manipulator/robot.xacro (robot description, xacro)
@@ -1,7 +1,7 @@
 <?xml version="1.0"?>
 <robot xmlns:xacro="http://www.ros.org/wiki/xacro" name="qm">
-    <!-- qudraputed -->
+    <!-- quadruped -->
     <xacro:arg name="robot_type" default="aliengo"/>
-    <xacro:include filename="$(find qm_description)/urdf/qudraputed/robot.xacro" />
+    <xacro:include filename="$(find qm_description)/urdf/quadruped/robot.xacro" />
     <!-- manipulatior -->
     <xacro:include filename="$(find qm_description)/urdf/manipulator/j2n6s300fix.xacro"/>
@@ -13,4 +13,6 @@
     </joint>
     <xacro:j2n6s300  base_parent="arm_base_link"/>
+    <!-- sensor -->
+    <xacro:include filename="$(find qm_description)/urdf/sensor/ft_sensor.xacro"/>
     <!-- ros_control plugin -->
     <gazebo>
@@ -18,5 +20,5 @@
             <robotNamespace>/</robotNamespace>
             <robotParam>qm_description</robotParam>
-            <robotSimType>qm_gazebo/DogHwSim</robotSimType>
+            <robotSimType>qm_gazebo/QMHWSim</robotSimType>
         </plugin>
     </gazebo>

File: qm_description/urdf/quadruped_manipulator/robot_mpc.xacro (robot description, xacro)
@@ -1,7 +1,7 @@
 <?xml version="1.0"?>
 <robot xmlns:xacro="http://www.ros.org/wiki/xacro" name="qm">
-    <!-- qudraputed -->
+    <!-- quadruped -->
     <xacro:arg name="robot_type" default="aliengo"/>
-    <xacro:include filename="$(find qm_description)/urdf/qudraputed/robot.xacro" />
+    <xacro:include filename="$(find qm_description)/urdf/quadruped/robot.xacro" />
     <!-- manipulatior -->
     <xacro:include filename="$(find qm_description)/urdf/manipulator/j2n6s300fix.xacro"/>
@@ -13,6 +13,4 @@
     </joint>
     <xacro:j2n6s300  base_parent="arm_base_link"/>
-    <!-- sensor -->
-    <xacro:include filename="$(find qm_description)/urdf/sensor/ft_sensor.xacro"/>
     <!-- ros_control plugin -->
     <gazebo>
@@ -20,5 +18,5 @@
             <robotNamespace>/</robotNamespace>
             <robotParam>qm_description</robotParam>
-            <robotSimType>qm_gazebo/QMHWSim</robotSimType>
+            <robotSimType>qm_gazebo/DogHwSim</robotSimType>
         </plugin>
     </gazebo>

File: qm_description/urdf/sensor/ft_sensor.xacro (robot description, xacro)
@@ -8,18 +8,18 @@
             <origin xyz="0.0 0.0 0.0" rpy="0.0 0.0 0.0"/>
         </visual>
-        <!-- <collision>
+        <collision>
             <geometry>
                 <cylinder radius="0.0375" length="0.01"/>
             </geometry>
             <origin xyz="0.0 0.0 0.0" rpy="0.0 0.0 0.0"/>
-        </collision> -->
+        </collision>
         <inertial>
             <mass value="0.0001"/>
-            <inertia ixx="3.5989583333333335E-8"
-                     ixy="0.0"
-                     ixz="0.0"
-                     iyy="3.5156250000041194E-8"
-                     iyz="0.0"
-                     izz="7.03125E-8"/>
+            <inertia ixx="10"
+                     ixy="10"
+                     ixz="10"
+                     iyy="10"
+                     iyz="10"
+                     izz="10"/>
         </inertial>
         <!-- <inertial>
